Commit message: NTP 동기화, RF2O 설정 수정, DWB 파라미터 수정

File: src/jupiter_description/urdf/jupiter_astra.urdf (robot description, URDF)
Before this commit: robot jupiter_description, 12 links, 11 joints
Joints:
- joint base_joint: child base_link -> base_footprint; origin xyz=0.0 0.0 0.08 rpy=0 0 0 -> xyz=0.0 0.0 -0.08 rpy=0 0 0; parent base_footprint -> base_link

File: src/jupiter_description/urdf/jupiter_simple.urdf (robot description, URDF)
Before this commit: robot jupiter_simple, 7 links, 6 joints
Links:
- link camera_link: mass 0.03 -> 0.07; geometry collision box size=0.0258 0.09 0.025; visual box size=0.0258 0.09 0.025
Joints:
- joint camera_joint: origin xyz=0.08 0 0.10403 rpy=0 0 -0.05 -> xyz=0.274 0 0.055 rpy=0 0 0
- joint laser_joint: origin xyz=-0.03 0 0.13 rpy=0 0 0 -> xyz=-0.03 0 0.13 rpy=0 0 3.14159
